File: HW/PiFinder.sch (KiCad schematic (older format))
At the start: 8 parts, among them P1 CONN_01X05, U1 VL53L0X

Commit message: Finalized the design. Ready to order.
Parts:
- U1: footprint KicadLibrary:VL53L0x -> KicadFootprint:VL53L0x
Changed lines of the file:
@@
 F 0 "U1" H 5700 2400 60  0000 C CNN
 F 1 "VL53L0X" H 5700 3600 60  0000 C CNN
-F 2 "KicadLibrary:VL53L0x" H 5750 3150 60  0001 C CNN
+F 2 "KicadFootprint:VL53L0x" H 5750 3150 60  0001 C CNN
 F 3 "" H 5750 3150 60  0001 C CNN
 	1    5750 3150

Commit message: Updated the part numbers.
Parts:
- C1: PartNum (none) -> CL21B104MBCNNNC
- C2: PartNum (none) -> CL21A475KQFNNNG
- R1, R3: PartNum (none) -> MCR10ERTJ432
- R2, R4: PartNum (none) -> MCR10FZPJ103
- U1: PartNum (none) -> VL53L0CXV0DH/1
Changed lines of the file:
@@
 F 2 "KicadFootprint:VL53L0x" H 5750 3150 60  0001 C CNN
 F 3 "" H 5750 3150 60  0001 C CNN
+F 4 "VL53L0CXV0DH/1" H 5750 3150 60  0001 C CNN "PartNum"
 	1    5750 3150
 	1    0    0    -1
@@
 F 2 "Resistors_SMD:R_0805" V 4480 2450 50  0001 C CNN
 F 3 "" H 4550 2450 50  0000 C CNN
+F 4 "MCR10ERTJ432" V 4550 2450 60  0001 C CNN "PartNum"
 	1    4550 2450
 	1    0    0    -1
@@
 F 2 "Resistors_SMD:R_0805" V 4230 2450 50  0001 C CNN
 F 3 "" H 4300 2450 50  0000 C CNN
+F 4 "MCR10ERTJ432" V 4300 2450 60  0001 C CNN "PartNum"
 	1    4300 2450
 	1    0    0    -1
@@
 F 2 "Capacitors_SMD:C_0805" H 6738 3000 50  0001 C CNN
 F 3 "" H 6700 3150 50  0000 C CNN
+F 4 "CL21B104MBCNNNC" H 6700 3150 60  0001 C CNN "PartNum"
 	1    6700 3150
 	1    0    0    -1
@@
 F 2 "Capacitors_SMD:C_0805" H 7088 3000 50  0001 C CNN
 F 3 "" H 7050 3150 50  0000 C CNN
+F 4 "CL21A475KQFNNNG" H 7050 3150 60  0001 C CNN "PartNum"
 	1    7050 3150
 	1    0    0    -1
@@
 F 2 "Resistors_SMD:R_0805" V 4530 3900 50  0001 C CNN
 F 3 "" H 4600 3900 50  0000 C CNN
+F 4 "MCR10FZPJ103" V 4600 3900 60  0001 C CNN "PartNum"
 	1    4600 3900
 	1    0    0    -1
@@
 F 2 "Resistors_SMD:R_0805" V 4330 3900 50  0001 C CNN
 F 3 "" H 4400 3900 50  0000 C CNN
+F 4 "MCR10FZPJ103" V 4400 3900 60  0001 C CNN "PartNum"
 	1    4400 3900
 	1    0    0    -1
